File: Hardware/YNXT-WM01.sch (KiCad schematic (older format))
At the start: 45 parts, among them P1 USB_C_Plug, Q1 Q_NMOS_DGS, Q2 Q_NPN_BCE, SW1 SW_Push, U1 LTC4054ES5-4.2, U2 FS8205A, U3 DW01A, U4 E18-MS1-PCB, U5 STI3408B

Commit message: Add reset volume for each channel, edit scheme elements values
Parts:
- Q2: value Q_NPN_BCE -> C1815
- R2: value 1.65k -> 1.5k
- R3, R4: value 500 -> 470
Changed lines of the file:
@@
 P 2400 1550
 F 0 "R3" H 2250 1600 50  0000 L CNN
-F 1 "500" H 2200 1500 50  0000 L CNN
+F 1 "470" H 2200 1500 50  0000 L CNN
 F 2 "Resistor_SMD:R_0603_1608Metric" V 2330 1550 50  0001 C CNN
 F 3 "~" H 2400 1550 50  0001 C CNN
@@
 P 2400 2100
 F 0 "R2" H 2470 2146 50  0000 L CNN
-F 1 "1.65k" H 2470 2055 50  0000 L CNN
+F 1 "1.5k" H 2470 2055 50  0000 L CNN
 F 2 "Resistor_SMD:R_0603_1608Metric" V 2330 2100 50  0001 C CNN
 F 3 "~" H 2400 2100 50  0001 C CNN
@@
 P 850 6100
 F 0 "R4" H 700 6150 50  0000 L CNN
-F 1 "500" H 650 6050 50  0000 L CNN
+F 1 "470" H 650 6050 50  0000 L CNN
 F 2 "Resistor_SMD:R_0603_1608Metric" V 780 6100 50  0001 C CNN
 F 3 "~" H 850 6100 50  0001 C CNN
@@
 P 10250 5750
 F 0 "Q2" H 10441 5796 50  0000 L CNN
-F 1 "Q_NPN_BCE" H 10441 5705 50  0000 L CNN
+F 1 "C1815" H 10441 5705 50  0000 L CNN
 F 2 "Package_TO_SOT_SMD:SOT-23" H 10450 5850 50  0001 C CNN
 F 3 "~" H 10250 5750 50  0001 C CNN
